Commit message: launch rviz working

File: urdf/poppy.ros2_control.xacro (robot description, xacro)
@@ -7,5 +7,5 @@
         <param name="usb_port">/dev/ttyACM0</param>
         <param name="baud_rate">115200</param>
-        <!-- <param name="use_dummy">true</param> -->
+        <param name="use_dummy">true</param>
       </hardware>
       <joint name="m1">

File: urdf/poppy.xacro (robot description, xacro)
@@ -3,4 +3,11 @@
 <!-- Import Rviz colors -->
 <xacro:include filename="$(find poppy_description)/urdf/poppy.material.xacro" />
+<xacro:macro name="poppy" params="parent *origin">
+  <joint name="origin_to_link1" type="fixed">
+    <xacro:insert_block name="origin" />
+    <parent link="${parent}" />
+    <child link="base_link" />
+    <axis xyz="0 0 1" />
+  </joint>
 <!-- Base link -->
   <link name="base_link">
@@ -10,5 +17,5 @@
         <mesh filename="package://poppy_description/meshes/base.dae" />
       </geometry>
-      <material name="darkgrey">
+      <material name="darkgrey"/>
     </visual>
     <collision>
@@ -25,5 +32,5 @@
     <child link="link1" />
     <axis xyz="0 0 1" />
-	<limit velocity="4.8" effort="1" lower="-1.57" upper="1.57" />
+    <limit velocity="4.8" effort="1" lower="-1.57" upper="1.57" />
   </joint>
 <!-- Link 1 -->
@@ -34,5 +41,5 @@
         <mesh filename="package://poppy_description/meshes/long_U.dae" />
       </geometry>
-      <material name="darkgrey">
+      <material name="darkgrey"/>
     </visual>
     <collision>
@@ -53,5 +60,5 @@
     <child link="link2" />
     <axis xyz="0 0 -1" />
-	<limit velocity="4.8" effort="1" lower="-1.57" upper="1.57" />
+    <limit velocity="4.8" effort="1" lower="-1.57" upper="1.57" />
   </joint>
 <!-- link2 -->
@@ -62,5 +69,5 @@
         <mesh filename="package://poppy_description/meshes/section_1.dae" />
       </geometry>
-      <material name="darkgrey">
+      <material name="darkgrey"/>
     </visual>
     <collision>
@@ -81,5 +88,5 @@
     <child link="link3" />
     <axis xyz="0 0 -1" />
-	<limit velocity="4.8" effort="1" lower="-1.57" upper="1.57" />
+    <limit velocity="4.8" effort="1" lower="-1.57" upper="1.57" />
   </joint>
 <!-- link3 -->
@@ -90,5 +97,5 @@
         <mesh filename="package://poppy_description/meshes/section_2.dae" />
       </geometry>
-      <material name="darkgrey">
+      <material name="darkgrey"/>
     </visual>
     <collision>
@@ -103,5 +110,5 @@
     </inertial>
   </link>
- <!-- Motor 4 -->
+<!-- Motor 4 -->
   <joint name="m4" type="revolute">
     <origin xyz="0.045 0 0" rpy="0 -1.5707963267949 0" />
@@ -109,7 +116,7 @@
     <child link="link4" />
     <axis xyz="0 0 -1" />
-	<limit velocity="4.8" effort="1" lower="-1.57" upper="1.57" />
-  </joint>
- <!-- link4 -->
+    <limit velocity="4.8" effort="1" lower="-1.57" upper="1.57" />
+  </joint>
+<!-- link4 -->
   <link name="link4">
     <visual>
@@ -118,5 +125,5 @@
         <mesh filename="package://poppy_description/meshes/section_3.dae" />
       </geometry>
-      <material name="darkgrey">
+      <material name="darkgrey"/>
     </visual>
     <collision>
@@ -131,11 +138,11 @@
     </inertial>
   </link>
- <!-- Motor 5 -->
- <joint name="m5" type="revolute">
+<!-- Motor 5 -->
+  <joint name="m5" type="revolute">
     <origin xyz="0 -0.048 0" rpy="0 -1.5707963267949 0" />
     <parent link="link4" />
     <child link="link5" />
     <axis xyz="0 0 1" />
-	<limit velocity="4.8" effort="1" lower="-1.57" upper="1.57" />
+    <limit velocity="4.8" effort="1" lower="-1.57" upper="1.57" />
   </joint>
 <!-- link5 -->
@@ -146,5 +153,5 @@
         <mesh filename="package://poppy_description/meshes/section_4.dae" />
       </geometry>
-      <material name="darkgrey">
+      <material name="darkgrey"/>
     </visual>
     <collision>
@@ -163,17 +170,17 @@
   <link name="gripper">
     <visual>
-	  <origin xyz="0 0 0" rpy="0 0 0" />
-	  <geometry>
-	    <mesh filename="package://poppy_description/meshes/gripper.dae" />
-	  </geometry>
-	  <material name="darkgrey">
-    </visual>
-    <collision>
-	  <origin xyz="0 -0.04 0" rpy="-1.5707963267949 0 0" />
-	  <geometry>
-	    <cylinder length="0.06" radius="0.02" />
-	  </geometry>
-    </collision>
-	<inertial>
+      <origin xyz="0 0 0" rpy="0 0 0" />
+      <geometry>
+      <mesh filename="package://poppy_description/meshes/gripper.dae" />
+      </geometry>
+      <material name="darkgrey"/>
+    </visual>
+    <collision>
+      <origin xyz="0 -0.04 0" rpy="-1.5707963267949 0 0" />
+      <geometry>
+        <cylinder length="0.06" radius="0.02" />
+      </geometry>
+    </collision>
+    <inertial>
       <mass value="0.1" />
       <inertia ixx="0.03" iyy="0.03" izz="0.03" ixy="0.0" ixz="0.0" iyz="0.0" />
@@ -186,4 +193,5 @@
     <parent link="link5" />
     <child link="gripper" />
+    <limit velocity="4.8" effort="1" lower="-1.57" upper="1.57" />
   </joint>
 <!-- Moving tip of gripper -->
@@ -194,3 +202,4 @@
     <child link="moving_tip" />
   </joint>
+</xacro:macro>
 </robot>

Commit message: almost working

File: urdf/poppy.ros2_control.xacro (robot description, xacro)
@@ -6,11 +6,11 @@
         <plugin>dynamixel_hardware/DynamixelHardware</plugin>
         <param name="usb_port">/dev/ttyACM0</param>
-        <param name="baud_rate">115200</param>
-        <param name="use_dummy">true</param>
+        <param name="baud_rate">9600</param>
+        <!--<param name="use_dummy">true</param>-->
       </hardware>
       <joint name="m1">
         <param name="id">1</param>
         <command_interface name="position"/>
-        <command_interface name="velocity"/>
+        <!--command_interface name="velocity"/-->
         <state_interface name="position"/>
         <state_interface name="velocity"/>
@@ -20,5 +20,5 @@
         <param name="id">2</param>
         <command_interface name="position"/>
-        <command_interface name="velocity"/>
+        <!--command_interface name="velocity"/-->
         <state_interface name="position"/>
         <state_interface name="velocity"/>
@@ -28,5 +28,5 @@
         <param name="id">3</param>
         <command_interface name="position"/>
-        <command_interface name="velocity"/>
+        <!--command_interface name="velocity"/-->
         <state_interface name="position"/>
         <state_interface name="velocity"/>
@@ -36,5 +36,5 @@
         <param name="id">4</param>
         <command_interface name="position"/>
-        <command_interface name="velocity"/>
+        <!--command_interface name="velocity"/-->
         <state_interface name="position"/>
         <state_interface name="velocity"/>
@@ -44,5 +44,5 @@
         <param name="id">5</param>
         <command_interface name="position"/>
-        <command_interface name="velocity"/>
+        <!--command_interface name="velocity"/-->
         <state_interface name="position"/>
         <state_interface name="velocity"/>
@@ -52,5 +52,5 @@
         <param name="id">6</param>
         <command_interface name="position"/>
-        <command_interface name="velocity"/>
+        <!--command_interface name="velocity"/-->
         <state_interface name="position"/>
         <state_interface name="velocity"/>

File: urdf/poppy.xacro (robot description, xacro)
@@ -32,5 +32,5 @@
     <child link="link1" />
     <axis xyz="0 0 1" />
-    <limit velocity="4.8" effort="1" lower="-1.57" upper="1.57" />
+    <limit velocity="0.5" effort="0.3" lower="${-90*(pi/180)}" upper="${90*(pi/180)}" />
   </joint>
 <!-- Link 1 -->
@@ -60,5 +60,5 @@
     <child link="link2" />
     <axis xyz="0 0 -1" />
-    <limit velocity="4.8" effort="1" lower="-1.57" upper="1.57" />
+    <limit velocity="0.5" effort="0.3" lower="${-90*(pi/180)}" upper="${90*(pi/180)}" />
   </joint>
 <!-- link2 -->
@@ -88,5 +88,5 @@
     <child link="link3" />
     <axis xyz="0 0 -1" />
-    <limit velocity="4.8" effort="1" lower="-1.57" upper="1.57" />
+    <limit velocity="0.5" effort="0.3" lower="${-90*(pi/180)}" upper="${90*(pi/180)}" />
   </joint>
 <!-- link3 -->
@@ -116,5 +116,5 @@
     <child link="link4" />
     <axis xyz="0 0 -1" />
-    <limit velocity="4.8" effort="1" lower="-1.57" upper="1.57" />
+    <limit velocity="0.5" effort="0.3" lower="${-90*(pi/180)}" upper="${90*(pi/180)}" />
   </joint>
 <!-- link4 -->
@@ -144,5 +144,5 @@
     <child link="link5" />
     <axis xyz="0 0 1" />
-    <limit velocity="4.8" effort="1" lower="-1.57" upper="1.57" />
+    <limit velocity="0.5" effort="0.3" lower="${-90*(pi/180)}" upper="${90*(pi/180)}" />
   </joint>
 <!-- link5 -->
@@ -193,5 +193,5 @@
     <parent link="link5" />
     <child link="gripper" />
-    <limit velocity="4.8" effort="1" lower="-1.57" upper="1.57" />
+    <limit velocity="0.5" effort="0.3" lower="${-20*(pi/180)}" upper="${60*(pi/180)}" />
   </joint>
 <!-- Moving tip of gripper -->

Commit message: Rviz working, txrx problem pesists

File: urdf/poppy.ros2_control.xacro (robot description, xacro)
@@ -6,54 +6,54 @@
         <plugin>dynamixel_hardware/DynamixelHardware</plugin>
         <param name="usb_port">/dev/ttyACM0</param>
-        <param name="baud_rate">9600</param>
+        <param name="baud_rate">115200</param>
         <!--<param name="use_dummy">true</param>-->
       </hardware>
       <joint name="m1">
         <param name="id">1</param>
-        <command_interface name="position"/>
-        <!--command_interface name="velocity"/-->
+        <command_interface name="position" initial_value="512" />
+        <!--command_interface name="velocity" initial_value="0.05" /-->
         <state_interface name="position"/>
-        <state_interface name="velocity"/>
-        <state_interface name="effort"/>
+        <!--state_interface name="velocity"/-->
+        <!-- state_interface name="effort"/-->
       </joint>
       <joint name="m2">
         <param name="id">2</param>
-        <command_interface name="position"/>
-        <!--command_interface name="velocity"/-->
+        <command_interface name="position" />
+        <!--command_interface name="velocity" initial_value="0.05" /-->
         <state_interface name="position"/>
-        <state_interface name="velocity"/>
-        <state_interface name="effort"/>
+        <!--state_interface name="velocity"/-->
+        <!-- state_interface name="effort"/-->
       </joint>
       <joint name="m3">
         <param name="id">3</param>
-        <command_interface name="position"/>
-        <!--command_interface name="velocity"/-->
+        <command_interface name="position" />
+        <!--command_interface name="velocity" initial_value="0.05" /-->
         <state_interface name="position"/>
-        <state_interface name="velocity"/>
-        <state_interface name="effort"/>
+        <!--state_interface name="velocity"/-->
+        <!-- state_interface name="effort"/-->
       </joint>
       <joint name="m4">
         <param name="id">4</param>
-        <command_interface name="position"/>
-        <!--command_interface name="velocity"/-->
+        <command_interface name="position" />
+        <!--command_interface name="velocity" initial_value="0.05" /-->
         <state_interface name="position"/>
-        <state_interface name="velocity"/>
-        <state_interface name="effort"/>
+        <!--state_interface name="velocity"/-->
+        <!-- state_interface name="effort"/-->
       </joint>
       <joint name="m5">
         <param name="id">5</param>
-        <command_interface name="position"/>
-        <!--command_interface name="velocity"/-->
+        <command_interface name="position" />
+        <!--command_interface name="velocity" initial_value="0.05" /-->
         <state_interface name="position"/>
-        <state_interface name="velocity"/>
-        <state_interface name="effort"/>
+        <!--state_interface name="velocity"/-->
+        <!-- state_interface name="effort"/-->
       </joint>
 	  <joint name="m6">
         <param name="id">6</param>
-        <command_interface name="position"/>
-        <!--command_interface name="velocity"/-->
+        <command_interface name="position" />
+        <!--command_interface name="velocity" initial_value="0.05" /-->
         <state_interface name="position"/>
-        <state_interface name="velocity"/>
-        <state_interface name="effort"/>
+        <!--state_interface name="velocity"/-->
+        <!-- state_interface name="effort"/-->
       </joint>
     </ros2_control>

File: urdf/poppy.xacro (robot description, xacro)
@@ -32,5 +32,5 @@
     <child link="link1" />
     <axis xyz="0 0 1" />
-    <limit velocity="0.5" effort="0.3" lower="${-90*(pi/180)}" upper="${90*(pi/180)}" />
+    <limit velocity="1" effort="0.3" lower="${-150*(pi/180)}" upper="${150*(pi/180)}" />
   </joint>
 <!-- Link 1 -->
@@ -60,5 +60,5 @@
     <child link="link2" />
     <axis xyz="0 0 -1" />
-    <limit velocity="0.5" effort="0.3" lower="${-90*(pi/180)}" upper="${90*(pi/180)}" />
+    <limit velocity="1" effort="0.3" lower="${-150*(pi/180)}" upper="${150*(pi/180)}" />
   </joint>
 <!-- link2 -->
@@ -88,5 +88,5 @@
     <child link="link3" />
     <axis xyz="0 0 -1" />
-    <limit velocity="0.5" effort="0.3" lower="${-90*(pi/180)}" upper="${90*(pi/180)}" />
+<limit velocity="1" effort="0.3" lower="${-150*(pi/180)}" upper="${150*(pi/180)}" />
   </joint>
 <!-- link3 -->
@@ -116,5 +116,5 @@
     <child link="link4" />
     <axis xyz="0 0 -1" />
-    <limit velocity="0.5" effort="0.3" lower="${-90*(pi/180)}" upper="${90*(pi/180)}" />
+<limit velocity="1" effort="0.3" lower="${-150*(pi/180)}" upper="${150*(pi/180)}" />
   </joint>
 <!-- link4 -->
@@ -144,5 +144,5 @@
     <child link="link5" />
     <axis xyz="0 0 1" />
-    <limit velocity="0.5" effort="0.3" lower="${-90*(pi/180)}" upper="${90*(pi/180)}" />
+<limit velocity="1" effort="0.3" lower="${-150*(pi/180)}" upper="${150*(pi/180)}" />
   </joint>
 <!-- link5 -->
@@ -193,5 +193,5 @@
     <parent link="link5" />
     <child link="gripper" />
-    <limit velocity="0.5" effort="0.3" lower="${-20*(pi/180)}" upper="${60*(pi/180)}" />
+    <limit velocity="1" effort="0.3" lower="${-150*(pi/180)}" upper="${150*(pi/180)}" />
   </joint>
 <!-- Moving tip of gripper -->

Commit message: Up and running

File: urdf/poppy.ros2_control.xacro (robot description, xacro)
@@ -5,5 +5,5 @@
       <hardware>
         <plugin>dynamixel_hardware/DynamixelHardware</plugin>
-        <param name="usb_port">/dev/ttyACM0</param>
+        <param name="usb_port">/dev/ttyUSB0</param>
         <param name="baud_rate">115200</param>
         <!--<param name="use_dummy">true</param>-->
@@ -11,49 +11,49 @@
       <joint name="m1">
         <param name="id">1</param>
-        <command_interface name="position" initial_value="512" />
-        <!--command_interface name="velocity" initial_value="0.05" /-->
+        <command_interface name="position" initial_value="0.0" />
+        <!--command_interface name="velocity"/-->
         <state_interface name="position"/>
-        <!--state_interface name="velocity"/-->
-        <!-- state_interface name="effort"/-->
+        <state_interface name="velocity"/>
+        <!--state_interface name="effort"/-->
       </joint>
       <joint name="m2">
         <param name="id">2</param>
-        <command_interface name="position" />
-        <!--command_interface name="velocity" initial_value="0.05" /-->
+        <command_interface name="position" initial_value="0.0" />
+        <!--command_interface name="velocity"/-->
         <state_interface name="position"/>
-        <!--state_interface name="velocity"/-->
-        <!-- state_interface name="effort"/-->
+        <state_interface name="velocity"/>
+        <!--state_interface name="effort"/-->
       </joint>
       <joint name="m3">
         <param name="id">3</param>
-        <command_interface name="position" />
-        <!--command_interface name="velocity" initial_value="0.05" /-->
+        <command_interface name="position" initial_value="0.0" />
+        <!--command_interface name="velocity"/-->
         <state_interface name="position"/>
-        <!--state_interface name="velocity"/-->
-        <!-- state_interface name="effort"/-->
+        <state_interface name="velocity"/>
+        <!--state_interface name="effort"/-->
       </joint>
       <joint name="m4">
         <param name="id">4</param>
-        <command_interface name="position" />
-        <!--command_interface name="velocity" initial_value="0.05" /-->
+        <command_interface name="position" initial_value="0.0" />
+        <!--command_interface name="velocity"/-->
         <state_interface name="position"/>
-        <!--state_interface name="velocity"/-->
-        <!-- state_interface name="effort"/-->
+        <state_interface name="velocity"/>
+        <!--state_interface name="effort"/-->
       </joint>
       <joint name="m5">
         <param name="id">5</param>
-        <command_interface name="position" />
-        <!--command_interface name="velocity" initial_value="0.05" /-->
+        <command_interface name="position" initial_value="0.0" />
+        <!--command_interface name="velocity"/-->
         <state_interface name="position"/>
-        <!--state_interface name="velocity"/-->
-        <!-- state_interface name="effort"/-->
+        <state_interface name="velocity"/>
+        <!--state_interface name="effort"/-->
       </joint>
-	  <joint name="m6">
+      <joint name="m6">
         <param name="id">6</param>
-        <command_interface name="position" />
-        <!--command_interface name="velocity" initial_value="0.05" /-->
+        <command_interface name="position" initial_value="0.0" />
+        <!--command_interface name="velocity"/-->
         <state_interface name="position"/>
-        <!--state_interface name="velocity"/-->
-        <!-- state_interface name="effort"/-->
+        <state_interface name="velocity"/>
+        <!--state_interface name="effort"/-->
       </joint>
     </ros2_control>

File: urdf/poppy.xacro (robot description, xacro)
@@ -32,5 +32,5 @@
     <child link="link1" />
     <axis xyz="0 0 1" />
-    <limit velocity="1" effort="0.3" lower="${-150*(pi/180)}" upper="${150*(pi/180)}" />
+    <limit velocity="10" effort="0.4" lower="${-150*(pi/180)}" upper="${150*(pi/180)}" />
   </joint>
 <!-- Link 1 -->
@@ -59,6 +59,6 @@
     <parent link="link1" />
     <child link="link2" />
-    <axis xyz="0 0 -1" />
-    <limit velocity="1" effort="0.3" lower="${-150*(pi/180)}" upper="${150*(pi/180)}" />
+    <axis xyz="0 0 1" />
+    <limit velocity="10" effort="0.4" lower="${-150*(pi/180)}" upper="${150*(pi/180)}" />
   </joint>
 <!-- link2 -->
@@ -87,6 +87,6 @@
     <parent link="link2" />
     <child link="link3" />
-    <axis xyz="0 0 -1" />
-<limit velocity="1" effort="0.3" lower="${-150*(pi/180)}" upper="${150*(pi/180)}" />
+    <axis xyz="0 0 1" />
+<limit velocity="10" effort="0.4" lower="${-150*(pi/180)}" upper="${150*(pi/180)}" />
   </joint>
 <!-- link3 -->
@@ -116,5 +116,5 @@
     <child link="link4" />
     <axis xyz="0 0 -1" />
-<limit velocity="1" effort="0.3" lower="${-150*(pi/180)}" upper="${150*(pi/180)}" />
+<limit velocity="10" effort="0.4" lower="${-150*(pi/180)}" upper="${150*(pi/180)}" />
   </joint>
 <!-- link4 -->
@@ -143,6 +143,6 @@
     <parent link="link4" />
     <child link="link5" />
-    <axis xyz="0 0 1" />
-<limit velocity="1" effort="0.3" lower="${-150*(pi/180)}" upper="${150*(pi/180)}" />
+    <axis xyz="0 0 -1" />
+<limit velocity="10" effort="0.4" lower="${-150*(pi/180)}" upper="${150*(pi/180)}" />
   </joint>
 <!-- link5 -->
@@ -190,8 +190,8 @@
   <joint name="m6" type="revolute">
     <origin xyz="0 -0.058 0" rpy="0 -1.5707963267949 0" />
-    <axis xyz="0 0 -1" />
+    <axis xyz="0 0 1" />
     <parent link="link5" />
     <child link="gripper" />
-    <limit velocity="1" effort="0.3" lower="${-150*(pi/180)}" upper="${150*(pi/180)}" />
+    <limit velocity="10" effort="0.4" lower="${-90*(pi/180)}" upper="${30*(pi/180)}" />
   </joint>
 <!-- Moving tip of gripper -->
