Commit message: Modified poppy.xacro to add a virtual link in fixed tip

File: urdf/poppy.xacro (robot description, xacro)
@@ -32,5 +32,5 @@
     <child link="link1" />
     <axis xyz="0 0 1" />
-    <limit velocity="10" effort="0.4" lower="${-150*(pi/180)}" upper="${150*(pi/180)}" />
+    <limit velocity="10" effort="1" lower="${-150*(pi/180)}" upper="${150*(pi/180)}" />
   </joint>
 <!-- Link 1 -->
@@ -60,5 +60,5 @@
     <child link="link2" />
     <axis xyz="0 0 1" />
-    <limit velocity="10" effort="0.4" lower="${-150*(pi/180)}" upper="${150*(pi/180)}" />
+    <limit velocity="10" effort="1" lower="${-150*(pi/180)}" upper="${150*(pi/180)}" />
   </joint>
 <!-- link2 -->
@@ -88,5 +88,5 @@
     <child link="link3" />
     <axis xyz="0 0 1" />
-<limit velocity="10" effort="0.4" lower="${-150*(pi/180)}" upper="${150*(pi/180)}" />
+<limit velocity="10" effort="1" lower="${-150*(pi/180)}" upper="${150*(pi/180)}" />
   </joint>
 <!-- link3 -->
@@ -116,5 +116,5 @@
     <child link="link4" />
     <axis xyz="0 0 -1" />
-<limit velocity="10" effort="0.4" lower="${-150*(pi/180)}" upper="${150*(pi/180)}" />
+<limit velocity="10" effort="1" lower="${-150*(pi/180)}" upper="${150*(pi/180)}" />
   </joint>
 <!-- link4 -->
@@ -144,5 +144,5 @@
     <child link="link5" />
     <axis xyz="0 0 -1" />
-<limit velocity="10" effort="0.4" lower="${-150*(pi/180)}" upper="${150*(pi/180)}" />
+<limit velocity="10" effort="1" lower="${-150*(pi/180)}" upper="${150*(pi/180)}" />
   </joint>
 <!-- link5 -->
@@ -193,5 +193,12 @@
     <parent link="link5" />
     <child link="gripper" />
-    <limit velocity="10" effort="0.4" lower="${-90*(pi/180)}" upper="${30*(pi/180)}" />
+    <limit velocity="10" effort="1" lower="${-90*(pi/180)}" upper="${30*(pi/180)}" />
+  </joint>
+<!--Fixed tip of gripper -->
+  <link name="fixed_tip" />
+  <joint name="tg" type="fixed">
+    <origin xyz="0 -0.052 0" rpy="-1.5707963267949 0 0" />
+    <parent link="link5" />
+    <child link="fixed_tip" />
   </joint>
 <!-- Moving tip of gripper -->

Commit message: modified poppy.xacro to have float integers, remove fixed link and tried implementing a fixed gripper link

File: urdf/poppy.xacro (robot description, xacro)
@@ -3,11 +3,4 @@
 <!-- Import Rviz colors -->
 <xacro:include filename="$(find poppy_description)/urdf/poppy.material.xacro" />
-<xacro:macro name="poppy" params="parent *origin">
-  <joint name="origin_to_link1" type="fixed">
-    <xacro:insert_block name="origin" />
-    <parent link="${parent}" />
-    <child link="base_link" />
-    <axis xyz="0 0 1" />
-  </joint>
 <!-- Base link -->
   <link name="base_link">
@@ -32,5 +25,5 @@
     <child link="link1" />
     <axis xyz="0 0 1" />
-    <limit velocity="10" effort="1" lower="${-150*(pi/180)}" upper="${150*(pi/180)}" />
+      <limit velocity="10.1" effort="1.0" lower="${-150*(pi/180)}" upper="${150*(pi/180)}" />
   </joint>
 <!-- Link 1 -->
@@ -60,5 +53,5 @@
     <child link="link2" />
     <axis xyz="0 0 1" />
-    <limit velocity="10" effort="1" lower="${-150*(pi/180)}" upper="${150*(pi/180)}" />
+      <limit velocity="10.1" effort="1.0" lower="${-150*(pi/180)}" upper="${150*(pi/180)}" />
   </joint>
 <!-- link2 -->
@@ -88,5 +81,5 @@
     <child link="link3" />
     <axis xyz="0 0 1" />
-<limit velocity="10" effort="1" lower="${-150*(pi/180)}" upper="${150*(pi/180)}" />
+      <limit velocity="10.1" effort="1.0" lower="${-150*(pi/180)}" upper="${150*(pi/180)}" />
   </joint>
 <!-- link3 -->
@@ -116,5 +109,5 @@
     <child link="link4" />
     <axis xyz="0 0 -1" />
-<limit velocity="10" effort="1" lower="${-150*(pi/180)}" upper="${150*(pi/180)}" />
+      <limit velocity="10.1" effort="1.0" lower="${-150*(pi/180)}" upper="${150*(pi/180)}" />
   </joint>
 <!-- link4 -->
@@ -144,5 +137,5 @@
     <child link="link5" />
     <axis xyz="0 0 -1" />
-<limit velocity="10" effort="1" lower="${-150*(pi/180)}" upper="${150*(pi/180)}" />
+  <limit velocity="10.1" effort="1.0" lower="${-150*(pi/180)}" upper="${150*(pi/180)}" />
   </joint>
 <!-- link5 -->
@@ -193,10 +186,10 @@
     <parent link="link5" />
     <child link="gripper" />
-    <limit velocity="10" effort="1" lower="${-90*(pi/180)}" upper="${30*(pi/180)}" />
+    <limit velocity="10.1" effort="1.0" lower="${-90*(pi/180)}" upper="${30*(pi/180)}" />
   </joint>
 <!--Fixed tip of gripper -->
   <link name="fixed_tip" />
   <joint name="tg" type="fixed">
-    <origin xyz="0 -0.052 0" rpy="-1.5707963267949 0 0" />
+    <origin xyz="0 -0.11 0" rpy="-1.5707963267949 0 0" />
     <parent link="link5" />
     <child link="fixed_tip" />

Commit message: current version of poppy description with virtual tip

File: urdf/poppy.xacro (robot description, xacro)
@@ -3,5 +3,12 @@
 <!-- Import Rviz colors -->
 <xacro:include filename="$(find poppy_description)/urdf/poppy.material.xacro" />
-<!-- Base link -->
+  <xacro:macro name="poppy" params="parent *origin">
+  <joint name="origin_to_link1" type="fixed">
+    <xacro:insert_block name="origin" />
+    <parent link="${parent}" />
+    <child link="base_link" />
+    <axis xyz="0 0 1" />
+  </joint>
+  <!-- Base link -->
   <link name="base_link">
     <visual>
@@ -19,5 +26,5 @@
     </collision>
   </link>
-<!-- Motor 1 -->
+  <!-- Motor 1 -->
   <joint name="m1" type="revolute">
     <origin xyz="0 0 0.0327993216120967" rpy="0 0 0" />
@@ -27,5 +34,5 @@
       <limit velocity="10.1" effort="1.0" lower="${-150*(pi/180)}" upper="${150*(pi/180)}" />
   </joint>
-<!-- Link 1 -->
+  <!-- Link 1 -->
   <link name="link1">
     <visual>
@@ -47,5 +54,5 @@
     </inertial>
   </link>
-<!-- Motor 2 -->
+  <!-- Motor 2 -->
   <joint name="m2" type="revolute">
     <origin xyz="0 0 0.0240006783879033" rpy="0 -1.5707963267949 0" />
@@ -55,5 +62,5 @@
       <limit velocity="10.1" effort="1.0" lower="${-150*(pi/180)}" upper="${150*(pi/180)}" />
   </joint>
-<!-- link2 -->
+  <!-- link2 -->
   <link name="link2">
     <visual>
@@ -75,5 +82,5 @@
     </inertial>
   </link>
-<!-- Motor 3 -->
+  <!-- Motor 3 -->
   <joint name="m3" type="revolute">
     <origin xyz="0.054 0 0" rpy="0 0 0" />
@@ -83,5 +90,5 @@
       <limit velocity="10.1" effort="1.0" lower="${-150*(pi/180)}" upper="${150*(pi/180)}" />
   </joint>
-<!-- link3 -->
+  <!-- link3 -->
   <link name="link3">
     <visual>
@@ -103,5 +110,5 @@
     </inertial>
   </link>
-<!-- Motor 4 -->
+  <!-- Motor 4 -->
   <joint name="m4" type="revolute">
     <origin xyz="0.045 0 0" rpy="0 -1.5707963267949 0" />
@@ -111,5 +118,5 @@
       <limit velocity="10.1" effort="1.0" lower="${-150*(pi/180)}" upper="${150*(pi/180)}" />
   </joint>
-<!-- link4 -->
+  <!-- link4 -->
   <link name="link4">
     <visual>
@@ -131,5 +138,5 @@
     </inertial>
   </link>
-<!-- Motor 5 -->
+    <!-- Motor 5 -->
   <joint name="m5" type="revolute">
     <origin xyz="0 -0.048 0" rpy="0 -1.5707963267949 0" />
@@ -139,5 +146,5 @@
   <limit velocity="10.1" effort="1.0" lower="${-150*(pi/180)}" upper="${150*(pi/180)}" />
   </joint>
-<!-- link5 -->
+  <!-- link5 -->
   <link name="link5">
     <visual>
@@ -160,5 +167,20 @@
     </inertial>
   </link>
-<!-- gripper -->
+  <!--Fixed tip -->
+  <joint name="t6g" type="fixed">
+    <origin xyz="0 -0.116 0" rpy="0 0 0" />
+    <parent link="link5" />
+    <child link="virtual_tip" />
+  </joint>
+  <link name="virtual_tip" />
+  <!-- gripper -->
+  <!-- Motor 6 -->
+  <joint name="m6" type="revolute">
+    <origin xyz="0 0.058 0" rpy="0 -1.5707963267949 0" />
+    <parent link="virtual_tip" />
+    <child link="gripper" />
+    <axis xyz="0 0 1" />
+    <limit velocity="10.1" effort="1.0" lower="${-90*(pi/180)}" upper="${25*(pi/180)}" />
+  </joint>
   <link name="gripper">
     <visual>
@@ -180,21 +202,5 @@
     </inertial>
   </link>
-<!-- Motor 6 -->
-  <joint name="m6" type="revolute">
-    <origin xyz="0 -0.058 0" rpy="0 -1.5707963267949 0" />
-    <axis xyz="0 0 1" />
-    <parent link="link5" />
-    <child link="gripper" />
-    <limit velocity="10.1" effort="1.0" lower="${-90*(pi/180)}" upper="${30*(pi/180)}" />
-  </joint>
-<!--Fixed tip of gripper -->
-  <link name="fixed_tip" />
-  <joint name="tg" type="fixed">
-    <origin xyz="0 -0.11 0" rpy="-1.5707963267949 0 0" />
-    <parent link="link5" />
-    <child link="fixed_tip" />
-  </joint>
-<!-- Moving tip of gripper -->
-  <link name="moving_tip" />
+  <!-- Moving tip of gripper -->
   <joint name="t7m" type="fixed">
     <origin xyz="0 -0.052 0" rpy="-1.5707963267949 0 0" />
@@ -202,4 +208,5 @@
     <child link="moving_tip" />
   </joint>
+  <link name="moving_tip" />
 </xacro:macro>
 </robot>
