Commit message: generated urdf

File: urdf/poppy.urdf (robot description, URDF)
Before this commit: robot None, 0 links, 0 joints
Links:
- added link base_link; collision cylinder length=0.03 radius=0.08; visual mesh filename=package://poppy_description/meshes/base.dae
- added link gripper, mass 0.1; collision cylinder length=0.06 radius=0.02; visual mesh filename=package://poppy_description/meshes/gripper.dae
- added link link1, mass 0.1; collision cylinder length=0.02 radius=0.02; visual mesh filename=package://poppy_description/meshes/long_U.dae
- added link link2, mass 0.1; collision cylinder length=0.05 radius=0.02; visual mesh filename=package://poppy_description/meshes/section_1.dae
- added link link3, mass 0.1; collision cylinder length=0.05 radius=0.02; visual mesh filename=package://poppy_description/meshes/section_2.dae
- added link link4, mass 0.1; collision cylinder length=0.05 radius=0.02; visual mesh filename=package://poppy_description/meshes/section_3.dae
- added link link5, mass 0.1; collision cylinder length=0.06 radius=0.02; visual mesh filename=package://poppy_description/meshes/section_4.dae
- added link moving_tip
- added link virtual_tip
- added link world
Joints:
- added joint m1: type revolute, parent base_link, child link1, origin xyz=0 0 0.0327993216120967 rpy=0 0 0, axis 0 0 1, limit lower=-2.6179938779914944 upper=2.6179938779914944 effort=1.0 velocity=10.1
- added joint m2: type revolute, parent link1, child link2, origin xyz=0 0 0.0240006783879033 rpy=0 -1.5707963267949 0, axis 0 0 1, limit lower=-2.6179938779914944 upper=2.6179938779914944 effort=1.0 velocity=10.1
- added joint m3: type revolute, parent link2, child link3, origin xyz=0.054 0 0 rpy=0 0 0, axis 0 0 1, limit lower=-2.6179938779914944 upper=2.6179938779914944 effort=1.0 velocity=10.1
- added joint m4: type revolute, parent link3, child link4, origin xyz=0.045 0 0 rpy=0 -1.5707963267949 0, axis 0 0 -1, limit lower=-2.6179938779914944 upper=2.6179938779914944 effort=1.0 velocity=10.1
- added joint m5: type revolute, parent link4, child link5, origin xyz=0 -0.048 0 rpy=0 -1.5707963267949 0, axis 0 0 -1, limit lower=-2.6179938779914944 upper=2.6179938779914944 effort=1.0 velocity=10.1
- added joint m6: type revolute, parent virtual_tip, child gripper, origin xyz=0 0.058 0 rpy=0 -1.5707963267949 0, axis 0 0 1, limit lower=-1.5707963267948966 upper=0.4363323129985824 effort=1.0 velocity=10.1
- added joint origin_to_link1: type fixed, parent world, child base_link, origin xyz=0 0 0 rpy=0 0 0, axis 0 0 1
- added joint t6g: type fixed, parent link5, child virtual_tip, origin xyz=0 -0.116 0 rpy=0 0 0
- added joint t7m: type fixed, parent gripper, child moving_tip, origin xyz=0 -0.052 0 rpy=-1.5707963267949 0 0
